Commit message: Major update: Kalman filter, adaptive threshold, persistent calibration
- Add Kalman filter for ball state estimation with adaptive R based on f_total
- Add adaptive threshold using configurable ref_roi brightness tracking (camera drift comp)
- Expand eef_pos_shm 6→9D (3 fingers × XYZ global frame)
- Remove f_res clamp (-30) to expose raw negative values for diagnostics
- Save/restore ref_baseline, ref_brightness, b_val across node restarts via JSON
- Unify adaptive threshold between calibration and operation nodes
- Add force_coeffs.json loading with hardcoded fallback
- Add show_gui launch parameter (DeclareLaunchArgument) for OpenCV windows
- Fix set_force_zero: remove warmup condition, persist b_val+brightness to JSON
- Add Clear All Data button to calibration UI
- Disable calibration buttons until Start/Resume Vision
- CSV: add f_exp, xyz_des_z, K_task, D_task, cop_raw, f_total, eef_vel, eef_cur, kf trace
- Remove 10s v4l2 camera settings re-apply (caused blackouts)
- Remove unused RViz2 from launch file

Co-Authored-By: Claude Opus 4.7 <noreply@anthropic.com>

File: src/torque_controller/urdf/hand_0926.urdf (robot description, URDF)
Before this commit: robot hand_0926, 16 links, 15 joints
Joints:
- joint F2EEF: origin xyz=-0.007 0.065 -0.02 rpy=0 0 0.785398 -> xyz=-0.007 0.065 -0.02 rpy=0 0 0.65
- joint F3EEF: origin xyz=-0.007 0.065 -0.02 rpy=0 0 0.82 -> xyz=-0.007 0.065 -0.02 rpy=0 0 0.785398
